File: hardware/BREAD_Slice.kicad_pcb (KiCad board)
At the start: 2 copper layers, 70 x 100 mm, 27 parts, among them J1 Conn_01x10_Female, J2 Screw_Terminal_01x02, J3 Screw_Terminal_01x02, Q1 IRLZ44N

Commit message: removed i2c conn silk
Other:
- board text removed: "5V I2C Connector"
Changed lines of the file:
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@@
 		(tags "Potentiometer vertical Bourns 3266W")
 		(property "Reference" "RV1"
-			(at -2.54 -2.27 360)
+			(at -2.54 -2.27 0)
 			(layer "F.SilkS")
 			(effects
@@
 		)
 		(property "Value" "100k"
-			(at -2.54 4.73 360)
+			(at -2.54 4.73 0)
 			(layer "F.Fab")
 			(effects
@@
 		)
 		(fp_text user "${REFERENCE}"
-			(at -3.175 1.23 360)
+			(at -3.175 1.23 0)
 			(layer "F.Fab")
 			(effects
@@
 		(tags "TO-220-3 Horizontal RM 2.54mm")
 		(property "Reference" "Q1"
-			(at 2.54 -20.58 360)
+			(at 2.54 -20.58 0)
 			(layer "F.SilkS")
 			(effects
@@
 		)
 		(property "Value" "IRLZ44N"
-			(at 2.54 2 360)
+			(at 2.54 2 0)
 			(layer "F.Fab")
 			(effects
@@
 		)
 		(fp_text user "${REFERENCE}"
-			(at 2.54 -20.58 360)
+			(at 2.54 -20.58 0)
 			(layer "F.Fab")
 			(effects
@@
 		(tags "capacitor")
 		(property "Reference" "C6"
-			(at 0 1.85 360)
+			(at 0 1.85 0)
 			(layer "B.SilkS")
 			(effects
@@
 		)
 		(property "Value" "1uF"
-			(at 0 -1.85 360)
+			(at 0 -1.85 0)
 			(layer "B.Fab")
 			(effects
@@
 		)
 		(fp_text user "${REFERENCE}"
-			(at 0 0 360)
+			(at 0 0 0)
 			(layer "B.Fab")
 			(effects
@@
 		(layer "B.SilkS")
 		(effects
-			(font
-				(size 1 1)
-				(thickness 0.15)
-			)
-			(justify bottom mirror)
-		)
-	)
-	(gr_text "5V I2C \nConnector"
-		(at 150.22 129.24 0)
-		(layer "B.SilkS")
-		(effects

Commit message: removed old
Parts:
- added NT1: NetTie_2, NetTie:NetTie-2_SMD_Pad2.0mm, B.Cu at (128.7, 115.2)
- C6: moved to F.Cu
- HS1, HS2: footprint KML-Custom:Thermal Pad -> kml-custom:Thermal Pad
- U1: value ~ -> AP63205
- moved C6 16.9 mm to (164.1, 84.4), turned to -90 degrees
- moved C5 15.0 mm to (178.1, 79.5), turned to -90 degrees
- moved Q1 13.4 mm to (161.2, 85.4), turned to 90 degrees
- moved D2 11.1 mm to (160.5, 73.4), turned to 180 degrees
- moved RV1 10.5 mm to (173.9, 92.0), turned to -135 degrees
- moved C7 10.3 mm to (178.3, 60.8)
- moved J3 9.98 mm to (188.2, 83.0)
- moved HS2 7.56 mm to (152.7, 82.8)
- moved R1 1.46 mm to (168.4, 76.0)
- moved L2 1.38 mm to (138.7, 55.3)
- moved G*** 1.05 mm to (174.7, 112.6)
- moved Logo1 0.65 mm to (128.2, 71.9)
- moved J2 0.30 mm to (188.3, 60.9), turned to 90 degrees
- moved C4 0.05 mm to (133.8, 116.4)
Connections:
- net /E_STOP renamed /ESTOP
- A1 pad 10: /D7 -> unconnected-(A1-D7-Pad10)
- A1 pad 11: /D8 -> unconnected-(A1-D8-Pad11)
- A1 pad 12: /D9 -> unconnected-(A1-D9-Pad12)
- A1 pad 13: /D10 -> unconnected-(A1-D10-Pad13)
- A1 pad 14: /D11 -> unconnected-(A1-D11-Pad14)
- A1 pad 15: /D12 -> unconnected-(A1-D12-Pad15)
- A1 pad 16: /D13 -> unconnected-(A1-D13-Pad16)
- A1 pad 18: /AREF -> unconnected-(A1-AREF-Pad18)
- A1 pad 20: /A1 -> unconnected-(A1-A1-Pad20)
- A1 pad 21: /A2 -> unconnected-(A1-A2-Pad21)
- A1 pad 22: /A3 -> unconnected-(A1-A3-Pad22)
- A1 pad 25: /A6 -> unconnected-(A1-A6-Pad25)
- A1 pad 26: /A7 -> unconnected-(A1-A7-Pad26)
- A1 pad 28: /RESET -> unconnected-(A1-~{RESET}-Pad28)
- C5 pad 2: GND -> GNDPWR
- C6 pad 2: GND -> GNDPWR
- C7 pad 2: GND -> GNDPWR
- D2 pad 2: GND -> GNDPWR
- J1 pad 1: GND -> GNDPWR
- J1 pad 10: GND -> GNDPWR
- J1 pad 5: GND -> GNDPWR
- J2 pad 2: GND -> GNDPWR
- J3 pad 1: GND -> GNDPWR
- RV1 pad 2: GND -> GNDPWR
- RV1 pad 3: GND -> GNDPWR
Routing:
- net GNDPWR: track 0.00 -> 45.0 mm, vias 0 -> 1
- net /Buck Conveter/out: track 69.4 -> 52.2 mm
- net /switching: track 53.9 -> 40.0 mm
- net /feedback: track 43.0 -> 50.2 mm
- net Net-(D2-K): track 29.7 -> 36.5 mm
- net /Buck Conveter/in: track 40.4 -> 36.9 mm
- net +12V: track 46.9 -> 48.2 mm, vias 1 -> 0
- net GND: track 17.7 -> 16.8 mm, vias 14 -> 20
- added copper zone on B.Cu, net GNDPWR
Other:
- outline, holes or cut-outs redrawn
- board text added: "BREAD Slice Buck Conv. SLC_BUCK R3 04-2025"
- board text removed: "+"
- board text removed: "BREAD Slice Buck Converter SLC_BUCK R2 04-2025"
- board text removed: "Vin"
- board text removed: "Vout"
