File: hardware-new/buck_conv.kicad_sch (KiCad schematic)
At the start: 9 parts, among them Q1 IRLZ44N

Commit message: finalized to 2L templ
Parts:
- HS2: footprint KML-Custom:Thermal Pad -> kml-custom:Thermal Pad
Changed lines of the file:
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@@
 		(instances
 			(project "BREAD_Slice"
-				(path "/66043bca-a260-4915-9fce-8a51d324c687/b645e956-7376-4c87-8c1d-444a21ed343a"
+				(path "/66043bca-a260-4915-9fce-8a51d324c687/bcddcbdb-40ba-43e9-ba1c-26ee4c61fa84"
 					(reference "C7")
 					(unit 1)
@@
 		(instances
 			(project "BREAD_Slice"
-				(path "/66043bca-a260-4915-9fce-8a51d324c687/b645e956-7376-4c87-8c1d-444a21ed343a"
+				(path "/66043bca-a260-4915-9fce-8a51d324c687/bcddcbdb-40ba-43e9-ba1c-26ee4c61fa84"
 					(reference "C6")
+					(unit 1)
+				)
+			)
+		)
+	)
+	(symbol
+		(lib_id "Mechanical:Heatsink_Pad")
+		(at 130.81 52.07 0)
+		(mirror y)
+		(unit 1)
+		(exclude_from_sim no)
+		(in_bom yes)
+		(on_board yes)
+		(dnp no)
+		(property "Reference" "HS2"
+			(at 127 50.1649 0)
+			(effects
+				(font
+					(size 1.27 1.27)
+				)
+				(justify left)
+			)
+		)
+		(property "Value" "Heatsink_Pad"
+			(at 127 52.7049 0)
+			(effects
+				(font
+					(size 1.27 1.27)
+				)
+				(justify left)
+			)
+		)
+		(property "Footprint" "kml-custom:Thermal Pad"
+			(at 130.5052 53.34 0)
+			(effects
+				(font
+					(size 1.27 1.27)
+				)
+				(hide yes)
+			)
+		)
+		(property "Datasheet" "~"
+			(at 130.5052 53.34 0)
+			(effects
+				(font
+					(size 1.27 1.27)
+				)
+				(hide yes)
+			)
+		)
+		(property "Description" "Heatsink with electrical connection, 1 pin"
+			(at 130.81 52.07 0)
+			(effects
+				(font
+					(size 1.27 1.27)
+				)
+				(hide yes)
+			)
+		)
+		(pin "1"
+		)
+		(instances
+			(project ""
+				(path "/66043bca-a260-4915-9fce-8a51d324c687/bcddcbdb-40ba-43e9-ba1c-26ee4c61fa84"
+					(reference "HS2")
 					(unit 1)
 				)
@@
 		)
 		(instances
-			(project ""
-				(path "/66043bca-a260-4915-9fce-8a51d324c687/b645e956-7376-4c87-8c1d-444a21ed343a"
+			(project "BREAD_Slice"
+				(path "/66043bca-a260-4915-9fce-8a51d324c687/bcddcbdb-40ba-43e9-ba1c-26ee4c61fa84"
 					(reference "Q1")
 					(unit 1)
@@
 		(instances
 			(project "BREAD_Slice"
-				(path "/66043bca-a260-4915-9fce-8a51d324c687/b645e956-7376-4c87-8c1d-444a21ed343a"
+				(path "/66043bca-a260-4915-9fce-8a51d324c687/bcddcbdb-40ba-43e9-ba1c-26ee4c61fa84"
 					(reference "R1")
 					(unit 1)
@@
 		(instances
 			(project "BREAD_Slice"
-				(path "/66043bca-a260-4915-9fce-8a51d324c687/b645e956-7376-4c87-8c1d-444a21ed343a"
+				(path "/66043bca-a260-4915-9fce-8a51d324c687/bcddcbdb-40ba-43e9-ba1c-26ee4c61fa84"
 					(reference "RV1")
 					(unit 1)
@@
 		)
 		(instances
-			(project ""
-				(path "/66043bca-a260-4915-9fce-8a51d324c687/b645e956-7376-4c87-8c1d-444a21ed343a"
+			(project "BREAD_Slice"
+				(path "/66043bca-a260-4915-9fce-8a51d324c687/bcddcbdb-40ba-43e9-ba1c-26ee4c61fa84"
 					(reference "L2")
 					(unit 1)
@@
 		(instances
 			(project "BREAD_Slice"
-				(path "/66043bca-a260-4915-9fce-8a51d324c687/b645e956-7376-4c87-8c1d-444a21ed343a"
+				(path "/66043bca-a260-4915-9fce-8a51d324c687/bcddcbdb-40ba-43e9-ba1c-26ee4c61fa84"
 					(reference "C5")
 					(unit 1)
@@
 		(instances
 			(project "BREAD_Slice"
-				(path "/66043bca-a260-4915-9fce-8a51d324c687/b645e956-7376-4c87-8c1d-444a21ed343a"
+				(path "/66043bca-a260-4915-9fce-8a51d324c687/bcddcbdb-40ba-43e9-ba1c-26ee4c61fa84"
 					(reference "D2")
 					(unit 1)
 				)
-			)
-		)
-	)
-	(symbol
-		(lib_id "Mechanical:Heatsink_Pad")
-		(at 130.81 52.07 0)
-		(mirror y)
-		(unit 1)
-		(exclude_from_sim yes)
-		(in_bom yes)
-		(on_board yes)
-		(dnp no)
-		(property "Reference" "HS2"
-			(at 127 50.1649 0)
-			(effects
-				(font
-					(size 1.27 1.27)
-				)
-				(justify left)
-			)
-		)
-		(property "Value" "Heatsink_Pad"
-			(at 127 52.7049 0)
-			(effects
-				(font
-					(size 1.27 1.27)
-				)
-				(justify left)
-			)
-		)
-		(property "Footprint" "KML-Custom:Thermal Pad"
-			(at 130.5052 53.34 0)
-			(effects
-				(font
-					(size 1.27 1.27)
-				)
-				(hide yes)
-			)
-		)
-		(property "Datasheet" "~"
-			(at 130.5052 53.34 0)
-			(effects
-				(font
-					(size 1.27 1.27)
-				)
-				(hide yes)
-			)
-		)
-		(property "Description" "Heatsink with electrical connection, 1 pin"
-			(at 130.81 52.07 0)
-			(effects
-				(font
-					(size 1.27 1.27)
-				)
-				(hide yes)
-			)
-		)
-		(pin "1"
-		)
-		(instances
-			(project ""
-				(path "/66043bca-a260-4915-9fce-8a51d324c687/b645e956-7376-4c87-8c1d-444a21ed343a"
-					(reference "HS2")
-					(unit 1)
-				)
